Commit message: training steps

File: Test_training/source/Test_training/Test_training/assets/robots/urdf/biped_s40.urdf (robot description, URDF)
Before this commit: robot my_robot_description, 49 links, 48 joints
Links:
- link zarm_l7_link: geometry collision box size=0.03 0.03 0.06; visual box size=0.03 0.03 0.06
- link zarm_r7_link: geometry collision box size=0.03 0.03 0.06; visual box size=0.03 0.03 0.06

Commit message: empty scene + fix position,eff

File: Test_training/source/Test_training/Test_training/assets/robots/urdf/biped_s40.urdf (robot description, URDF)
Before this commit: robot my_robot_description, 49 links, 48 joints
Links:
- link zarm_l_finger_left: geometry collision box size=0.12 0.035 0.035; visual box size=0.12 0.03 0.03
- link zarm_l_finger_right: geometry collision box size=0.12 0.035 0.035; visual box size=0.12 0.03 0.03
- link zarm_r7_end_effector: mass 0.2 -> 0.5
- link zarm_r7_link: mass 0.81 -> 1.2
- link zarm_r_finger_left: mass 0.05 -> 0.12; geometry collision box size=0.08 0.03 0.03; visual box size=0.08 0.03 0.03
- link zarm_r_finger_right: mass 0.05 -> 0.12; geometry collision box size=0.08 0.03 0.03; visual box size=0.08 0.03 0.03
Joints:
- joint zarm_r7_end_effector_joint: origin xyz=0 0 0 rpy=0 1.57079632679 0 -> xyz=0 0 0 rpy=0 0 0
- joint zarm_r7_joint: limit lower=-1.5707963267949 upper=1.5707963267949 effort=6.0 velocity=21.666 -> lower=-1.57079632679 upper=1.57079632679 effort=6.0 velocity=21.666
- joint zarm_r_finger_left_joint: origin xyz=-0.02 0.035 0 rpy=0 0 0 -> xyz=0 0.035 0 rpy=0 0 0
- joint zarm_r_finger_right_joint: origin xyz=-0.02 -0.035 0 rpy=0 0 0 -> xyz=0 -0.035 0 rpy=0 0 0
