Commit message: supported model

File: Test_training/source/Test_training/Test_training/assets/robots/urdf/supported_biped_s40.urdf (robot description, URDF)
Before this commit: robot my_robot_description, 49 links, 48 joints
Links:
- added link support_base, mass 0.2; collision box size=0.3 0.3 0.05; visual box size=0.3 0.3 0.05
- added link support_stick, mass 0.01; collision cylinder length=1.0 radius=0.01; visual cylinder length=1.0 radius=0.01
Joints:
- added joint robot_fixed_mount: type fixed, parent support_stick, child base_link, origin xyz=0 0 0 rpy=0 0 0
- added joint support_stick_joint: type fixed, parent support_base, child support_stick, origin xyz=0 0 0.05 rpy=0 0 0

Commit message: support model

File: Test_training/source/Test_training/Test_training/assets/robots/urdf/supported_biped_s40.urdf (robot description, URDF)
Before this commit: robot my_robot_description, 51 links, 50 joints
Links:
- link zarm_l6_link: geometry collision cylinder length=0.12 radius=0.025; visual cylinder length=0.12 radius=0.025
- link zarm_l7_link: geometry 
- link zarm_l_finger_left: geometry collision box size=0.12 0.02 0.02; visual box size=0.04 0.02 0.02
- link zarm_l_finger_right: geometry collision box size=0.12 0.035 0.035; visual box size=0.04 0.02 0.02
- link zarm_r6_link: geometry collision cylinder length=0.12 radius=0.025; visual cylinder length=0.12 radius=0.025
- link zarm_r7_end_effector: mass 0.5 -> 0.2
- link zarm_r7_link: mass 1.2 -> 0.81; geometry 
- link zarm_r_finger_left: mass 0.12 -> 0.05; geometry collision box size=0.12 0.02 0.02; visual box size=0.04 0.02 0.02
- link zarm_r_finger_right: mass 0.12 -> 0.05; geometry collision box size=0.12 0.035 0.035; visual box size=0.04 0.02 0.02
Joints:
- joint robot_fixed_mount: origin xyz=0 0 0 rpy=0 0 0 -> xyz=0 0 0.9 rpy=0 0 0
- joint zarm_r7_end_effector_joint: origin xyz=0 0 0 rpy=0 0 0 -> xyz=0 0 0 rpy=0 1.57079632679 0
- joint zarm_r7_joint: limit lower=-1.57079632679 upper=1.57079632679 effort=6.0 velocity=21.666 -> lower=-1.5707963267949 upper=1.5707963267949 effort=6.0 velocity=21.666
- joint zarm_r_finger_left_joint: origin xyz=0 0.035 0 rpy=0 0 0 -> xyz=-0.02 -0.035 0 rpy=0 0 0
- joint zarm_r_finger_right_joint: origin xyz=0 -0.035 0 rpy=0 0 0 -> xyz=-0.02 0.035 0 rpy=0 0 0

Commit message: updated usd, cameras

File: Test_training/source/Test_training/Test_training/assets/robots/urdf/supported_biped_s40.urdf (robot description, URDF)
Before this commit: robot my_robot_description, 51 links, 50 joints
Links:
- link l_foot_heel: geometry collision sphere radius=0.005; visual sphere radius=0.005
- link l_foot_toe: geometry collision sphere radius=0.005; visual sphere radius=0.005
- link ll_foot_heel: geometry collision sphere radius=0.005; visual sphere radius=0.005
- link ll_foot_toe: geometry collision sphere radius=0.005; visual sphere radius=0.005
- link lr_foot_heel: geometry collision sphere radius=0.005; visual sphere radius=0.005
- link lr_foot_toe: geometry collision sphere radius=0.005; visual sphere radius=0.005
- link r_foot_heel: geometry collision sphere radius=0.005; visual sphere radius=0.005
- link r_foot_toe: geometry collision sphere radius=0.005; visual sphere radius=0.005
- link rl_foot_heel: geometry collision sphere radius=0.005; visual sphere radius=0.005
- link rl_foot_toe: geometry collision sphere radius=0.005; visual sphere radius=0.005
- link rr_foot_heel: geometry collision sphere radius=0.005; visual sphere radius=0.005
- link rr_foot_toe: geometry collision sphere radius=0.005; visual sphere radius=0.005
- link zarm_l7_link: geometry collision box size=0.03 0.03 0.06; visual box size=0.03 0.03 0.06
- link zarm_r7_link: geometry collision box size=0.03 0.03 0.06; visual box size=0.03 0.03 0.06
Joints:
- removed joint camera_base
- added joint camera_base_joint: type fixed, parent zhead_2_link, child camera_base, origin xyz=0.0766792844154498 0 0.0571889355165869 rpy=0 0.610865238198013 0
