Commit message: s40_no_gripper model

File: Test_training/source/Test_training/Test_training/assets/robots/s40_full_arms/biped_s40/urdf/biped_s40_no_grippers.urdf (robot description, URDF)
Before this commit: robot biped_s40, 46 links, 45 joints
Links:
- link zarm_l7_end_effector: geometry 
- link zarm_l7_link: geometry visual mesh filename=../meshes/l_hand_roll_no_gripper.STL
- link zarm_r7_end_effector: geometry 
- link zarm_r7_link: geometry visual mesh filename=../meshes/r_hand_roll_no_gripper.STL
